File: sd-esd-rev1/sd-esd-rev1.kicad_pcb (KiCad board)
At the start: 2 copper layers, 53.7 x 25.4 mm, 12 parts, among them J10 2mm jumper, J11 WireTerm, J12 S3B-PH-K-S(LF)(SN), J4 CONN_10X2, J7 CONN_42.54_NOSILK

Commit message: Updated for kicad 6.0 https://www.kicad.org/blog/
Other:
- net class Default removed
- net class Power removed
- net class PwrMin removed
